File: Manual-Controller/st_pat_manual_ctrl_edits.sch (KiCad schematic (older format))
At the start: 15 parts, among them J4 BATTERY, SW1 SW_PWR, SW2 BTN_RST, SW3 BTN, SW4 BTN, SW5 BTN, U1 GPS_Breakout_746, U2 FEATHER_M0_BASIC_PROTO, U4 Sharp_Display_4694, U5 COTS_GPS_RECEIVER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

Commit message: added all the switches
Parts:
- added SW6, SW?: SW_DIP_x01, symbol Switch:SW_DIP_x01
- added SW7, SW8: BTN, Button_Switch_THT:SW_PUSH_6mm, symbol Switch:SW_Push
- SW2: value BTN_RST -> BTN
Connections:
- net BTN_A1: no longer SW5.1
- net BTN_A2: no longer SW4.1
- net BTN_A3: no longer SW3.1
- net GND: now also SW6.2, SW7.2, SW8.2, SW?.2
- net RST: no longer SW2.1
- new net BTN_PITCH+: SW2.1
- new net BTN_PITCH-: SW3.1
- new net BTN_ROLL+: SW4.1
- new net BTN_ROLL-: SW5.1
- new net BTN_YAW+: SW7.1
- new net BTN_YAW-: SW8.1
Other:
- note added: "BUTTON PADS FOR FLIGHT CONTROL"
- note added: "MANUAL <-> AUTOMATIC CONTROL"
- note added: "SAFETY KILL SWITCH (DROP IT LIKE IT'S HOT)"
- note removed: "BUTTONS - ALL OF THEM HAVE INTERNAL PULLUP"
- moved on the sheet: J4, SW1
Changed lines of the file:
@@
 encoding utf-8
 Sheet 1 1
-Title "ST_PAT SLIM"
+Title "ST_PATS2EB"
 Date "2021-02-05"
 Rev ""
@@
 L power:GND #PWR014
 U 1 1 60196448
-P 7250 5300
-F 0 "#PWR014" H 7250 5050 50  0001 C CNN
-F 1 "GND" H 7255 5127 50  0000 C CNN
-F 2 "" H 7250 5300 50  0001 C CNN
-F 3 "" H 7250 5300 50  0001 C CNN
-	1    7250 5300
-	1    0    0    -1
-$EndComp
-Wire Wire Line
-	7250 5300 7850 5300
+P 5650 5250
+F 0 "#PWR014" H 5650 5000 50  0001 C CNN
+F 1 "GND" H 5655 5077 50  0000 C CNN
+F 2 "" H 5650 5250 50  0001 C CNN
+F 3 "" H 5650 5250 50  0001 C CNN
+	1    5650 5250
+	1    0    0    -1
+$EndComp
+Wire Wire Line
+	5650 5250 6250 5250
 $Comp
 L power:+3V3 #PWR012
@@
 Text Notes 2550 1350 2    50   ~ 0
 GPS MODULE
-Text Notes 7900 4200 2    50   ~ 0
+Text Notes 6300 4150 2    50   ~ 0
 POWER SWITCH
 $Comp
@@
 	0    -1   -1   0
 $EndComp
-Text Notes 10600 4200 2    50   ~ 0
-BUTTONS - ALL OF THEM HAVE INTERNAL PULLUP
+Text Notes 10850 3400 2    50   ~ 0
+BUTTON PADS FOR FLIGHT CONTROL
 Text Label 9500 5800 2    50   ~ 0
-BTN_A1
+BTN_ROLL-
 Text Label 9500 5400 2    50   ~ 0
-BTN_A2
+BTN_ROLL+
 Text Label 9500 5000 2    50   ~ 0
-BTN_A3
+BTN_PITCH-
 Connection ~ 9900 5800
 Wire Wire Line
@@
 	1    0    0    -1
 $EndComp
-Connection ~ 9900 5400
 Wire Wire Line
 	9900 5400 9900 5800
@@
 $EndComp
 Text Label 9500 4600 2    50   ~ 0
-RST
+BTN_PITCH+
 Connection ~ 9900 5000
 Wire Wire Line
@@
 P 9700 4600
 F 0 "SW2" H 9700 4885 50  0000 C CNN
-F 1 "BTN_RST" H 9700 4794 50  0000 C CNN
+F 1 "BTN" H 9700 4794 50  0000 C CNN
 F 2 "Button_Switch_THT:SW_PUSH_6mm" H 9700 4800 50  0001 C CNN
 F 3 "~" H 9700 4800 50  0001 C CNN
@@
 L Switch:SW_Push_DPDT SW1
 U 1 1 602F6777
-P 7650 4900
-F 0 "SW1" H 7650 5385 50  0000 C CNN
-F 1 "SW_PWR" H 7650 5294 50  0000 C CNN
-F 2 "st_pat:SW_Rocker_A22K1H-EA" H 7650 5100 50  0001 C CNN
-F 3 "https://www.nkkswitches.com/pdf/ARockers-1.pdf" H 7650 5100 50  0001 C CNN
-	1    7650 4900
+P 6050 4850
+F 0 "SW1" H 6050 5335 50  0000 C CNN
+F 1 "SW_PWR" H 6050 5244 50  0000 C CNN
+F 2 "st_pat:SW_Rocker_A22K1H-EA" H 6050 5050 50  0001 C CNN
+F 3 "https://www.nkkswitches.com/pdf/ARockers-1.pdf" H 6050 5050 50  0001 C CNN
+	1    6050 4850
 	1    0    0    -1
 $EndComp
@@
 L Connector:Conn_01x02_Female J4
 U 1 1 601931F0
-P 8050 5200
-F 0 "J4" H 8078 5176 50  0000 L CNN
-F 1 "BATTERY" H 7750 5000 50  0000 L CNN
-F 2 "Connector_JST:JST_PH_S2B-PH-K_1x02_P2.00mm_Horizontal" H 8050 5200 50  0001 C CNN
-F 3 "~" H 8050 5200 50  0001 C CNN
-	1    8050 5200
-	1    0    0    -1
-$EndComp
-Wire Wire Line
-	7250 5100 7450 5100
+P 6450 5150
+F 0 "J4" H 6478 5126 50  0000 L CNN
+F 1 "BATTERY" H 6150 4950 50  0000 L CNN
+F 2 "Connector_JST:JST_PH_S2B-PH-K_1x02_P2.00mm_Horizontal" H 6450 5150 50  0001 C CNN
+F 3 "~" H 6450 5150 50  0001 C CNN
+	1    6450 5150
+	1    0    0    -1
+$EndComp
+Wire Wire Line
+	5650 5050 5850 5050
 $Comp
 L power:+BATT #PWR0101
 U 1 1 60232364
-P 7250 5100
-F 0 "#PWR0101" H 7250 4950 50  0001 C CNN
-F 1 "+BATT" H 7265 5273 50  0000 C CNN
-F 2 "" H 7250 5100 50  0001 C CNN
-F 3 "" H 7250 5100 50  0001 C CNN
-	1    7250 5100
-	1    0    0    -1
-$EndComp
-NoConn ~ 7450 4700
-NoConn ~ 7850 4600
-NoConn ~ 7850 4800
-NoConn ~ 7850 5000
+P 5650 5050
+F 0 "#PWR0101" H 5650 4900 50  0001 C CNN
+F 1 "+BATT" H 5665 5223 50  0000 C CNN
+F 2 "" H 5650 5050 50  0001 C CNN
+F 3 "" H 5650 5050 50  0001 C CNN
+	1    5650 5050
+	1    0    0    -1
+$EndComp
+NoConn ~ 5850 4650
+NoConn ~ 6250 4550
+NoConn ~ 6250 4750
+NoConn ~ 6250 4950
 $Comp
 L FEATHER_M0_BASIC_PROTO:FEATHER_M0_BASIC_PROTO U2
@@
 NoConn ~ 2850 4550
 NoConn ~ 1350 4550
+$Comp
+L Switch:SW_DIP_x01 SW6
+U 1 1 61985792
+P 8450 4550
+F 0 "SW6" H 8450 4817 50  0000 C CNN
+F 1 "SW_DIP_x01" H 8450 4726 50  0000 C CNN
+F 2 "" H 8450 4550 50  0001 C CNN
+F 3 "~" H 8450 4550 50  0001 C CNN
+	1    8450 4550
+	1    0    0    -1
+$EndComp
+Text Notes 7300 4150 0    50   ~ 0
+MANUAL <-> AUTOMATIC CONTROL
+Text Label 9500 4200 2    50   ~ 0
+BTN_YAW-
+Wire Wire Line
+	9900 4200 9900 4600
+$Comp
+L Switch:SW_Push SW8
+U 1 1 6199DAD0
+P 9700 4200
+F 0 "SW8" H 9700 4485 50  0000 C CNN
+F 1 "BTN" H 9700 4394 50  0000 C CNN
+F 2 "Button_Switch_THT:SW_PUSH_6mm" H 9700 4400 50  0001 C CNN
+F 3 "~" H 9700 4400 50  0001 C CNN
+	1    9700 4200
+	1    0    0    -1
+$EndComp
+Text Label 9500 3800 2    50   ~ 0
+BTN_YAW+
+Connection ~ 9900 4200
+Wire Wire Line
+	9900 3800 9900 4200
+$Comp
+L Switch:SW_Push SW7
+U 1 1 6199DADD
+P 9700 3800
+F 0 "SW7" H 9700 4085 50  0000 C CNN
+F 1 "BTN" H 9700 3994 50  0000 C CNN
+F 2 "Button_Switch_THT:SW_PUSH_6mm" H 9700 4000 50  0001 C CNN
+F 3 "~" H 9700 4000 50  0001 C CNN
+	1    9700 3800
+	1    0    0    -1
+$EndComp
+Connection ~ 9900 5400
+Connection ~ 9900 4600
+$Comp
+L Switch:SW_DIP_x01 SW?
+U 1 1 619B0937
+P 8450 5150
+F 0 "SW?" H 8450 5417 50  0000 C CNN
+F 1 "SW_DIP_x01" H 8450 5326 50  0000 C CNN
+F 2 "" H 8450 5150 50  0001 C CNN
+F 3 "~" H 8450 5150 50  0001 C CNN
+	1    8450 5150
+	1    0    0    -1
+$EndComp
+Wire Wire Line
+	8750 4550 8750 5150
+Connection ~ 8750 5150
+Text Notes 6950 4800 0    50   ~ 0
+SAFETY KILL SWITCH (DROP IT LIKE IT'S HOT)
+$Comp
+L power:GND #PWR0102
+U 1 1 6198A4F8
+P 8750 5350
+F 0 "#PWR0102" H 8750 5100 50  0001 C CNN
+F 1 "GND" H 8755 5177 50  0000 C CNN
+F 2 "" H 8750 5350 50  0001 C CNN
+F 3 "" H 8750 5350 50  0001 C CNN
+	1    8750 5350
+	1    0    0    -1
+$EndComp
+Wire Wire Line
+	8750 5150 8750 5350
+Wire Notes Line
+	3450 2750 7700 2750
 $EndSCHEMATC

Commit message: button header
Parts:
- removed D2: PWR_RED, LED_SMD:LED_1206_3216Metric_Pad1.42x1.75mm_HandSolder, symbol Device:LED
- removed D3: GEN_BLU, LED_SMD:LED_1206_3216Metric_Pad1.42x1.75mm_HandSolder, symbol Device:LED
- removed R2: 160, Resistor_SMD:R_0805_2012Metric_Pad1.20x1.40mm_HandSolder, symbol Device:R_US
- removed R3: 100, Resistor_SMD:R_0805_2012Metric_Pad1.20x1.40mm_HandSolder, symbol Device:R_US
- removed U2: FEATHER_M0_BASIC_PROTO, FEATHER_M0_BASIC_PROTO:FEATHER_M0_BASIC_PROTO, symbol FEATHER_M0_BASIC_PROTO:FEATHER_M0_BASIC_PROTO
- added J?: Conn_01x10_Female, symbol Connector:Conn_01x10_Female
- added U?: PIC18F26K83-canhw, symbol payload2022_custom:PIC18F26K83-canhw
- U1: symbol st_pat:GPS_Breakout_746 -> st_pat_manual_ctrl_edits-rescue:GPS_Breakout_746-st_pat
- U4: symbol st_pat:Sharp_Display_4694 -> st_pat_manual_ctrl_edits-rescue:Sharp_Display_4694-st_pat
- U5, U6: symbol st_pat:Telemetry_Breakout -> st_pat_manual_ctrl_edits-rescue:Telemetry_Breakout-st_pat
Connections:
- net BTN_PITCH+: now also J?.3 (Pin_3), U?.14 (RC3); no longer SW2.1
- net BTN_PITCH-: now also J?.4 (Pin_4), U?.15 (RC4); no longer SW3.1
- net BTN_ROLL+: now also J?.5 (Pin_5), U?.16 (RC5); no longer SW4.1
- net BTN_ROLL-: now also J?.6 (Pin_6), U?.17 (RC6); no longer SW5.1
- net BTN_YAW+: now also J?.1 (Pin_1), U?.12 (RC1); no longer SW7.1
- net BTN_YAW-: now also J?.2 (Pin_2), U?.13 (RC2); no longer SW8.1
- net MOSI: now also U4.4 (SCLK); no longer U4.5 (SI)
- net SCK: now also U4.2 (3v3); no longer U4.4 (SCLK)
- no-connect marks 19 -> 12
Other:
- note removed: "Estimate 50mA"
- note removed: "FEATHER M0 ADALOGGER"
- note removed: "P2_8 (D9) IS BATTERY MONITOR, DO NOT USE"
Changed lines of the file:
@@
 Text Notes 6300 4150 2    50   ~ 0
 POWER SWITCH
-$Comp
-L power:+BATT #PWR011
-U 1 1 6017627A
-P 6700 1600
-F 0 "#PWR011" H 6700 1450 50  0001 C CNN
-F 1 "+BATT" H 6500 1750 50  0000 L CNN
-F 2 "" H 6700 1600 50  0001 C CNN
-F 3 "" H 6700 1600 50  0001 C CNN
-	1    6700 1600
-	1    0    0    -1
-$EndComp
-$Comp
-L power:GND #PWR09
-U 1 1 60174E09
-P 6600 3550
-F 0 "#PWR09" H 6600 3300 50  0001 C CNN
-F 1 "GND" H 6700 3350 50  0000 R CNN
-F 2 "" H 6600 3550 50  0001 C CNN
-F 3 "" H 6600 3550 50  0001 C CNN
-	1    6600 3550
-	1    0    0    -1
-$EndComp
-$Comp
-L power:GND #PWR08
-U 1 1 60174547
-P 7450 2750
-F 0 "#PWR08" H 7450 2500 50  0001 C CNN
-F 1 "GND" H 7455 2577 50  0000 C CNN
-F 2 "" H 7450 2750 50  0001 C CNN
-F 3 "" H 7450 2750 50  0001 C CNN
-	1    7450 2750
-	1    0    0    -1
-$EndComp
-$Comp
-L power:+3V3 #PWR07
-U 1 1 60172EEF
-P 6850 1600
-F 0 "#PWR07" H 6850 1450 50  0001 C CNN
-F 1 "+3V3" H 6900 1750 50  0000 C CNN
-F 2 "" H 6850 1600 50  0001 C CNN
-F 3 "" H 6850 1600 50  0001 C CNN
-	1    6850 1600
-	1    0    0    -1
-$EndComp
-Text Label 6600 3150 0    50   ~ 0
-SHARP_CS_D5
-Text Label 6600 3050 0    50   ~ 0
-SHARP_DISP_D6
-Text Label 6600 2750 0    50   ~ 0
-GPS_FIX_D11
-Text Label 6600 2650 0    50   ~ 0
-GPS_PPS_D12
-Text Label 4200 1950 2    50   ~ 0
-RST
+Text Label 8650 2050 2    50   ~ 0
+SCK
 Text Label 8650 2200 2    50   ~ 0
-SCK
-Text Label 8650 2350 2    50   ~ 0
 MOSI
 Text Label 9600 2350 0    50   ~ 0
@@
 Text Label 9600 2050 0    50   ~ 0
 SHARP_DISP_D6
-Text Label 4200 2450 2    50   ~ 0
-BTN_A1
-Text Label 4200 2550 2    50   ~ 0
-BTN_A2
 Text Notes 1800 7100 2    50   ~ 0
 MAKES ERC HAPPY
@@
 	1    0    0    -1
 $EndComp
-$Comp
-L Device:LED D2
-U 1 1 6021AE05
-P 7000 1850
-F 0 "D2" H 7050 1750 50  0000 C CNN
-F 1 "PWR_RED" H 7100 2000 50  0000 C CNN
-F 2 "LED_SMD:LED_1206_3216Metric_Pad1.42x1.75mm_HandSolder" H 7000 1850 50  0001 C CNN
-F 3 "~" H 7000 1850 50  0001 C CNN
-	1    7000 1850
-	-1   0    0    1
-$EndComp
-$Comp
-L Device:R_US R2
-U 1 1 6021D72C
-P 7300 1850
-F 0 "R2" V 7400 1850 50  0000 C CNN
-F 1 "160" V 7186 1850 50  0000 C CNN
-F 2 "Resistor_SMD:R_0805_2012Metric_Pad1.20x1.40mm_HandSolder" V 7340 1840 50  0001 C CNN
-F 3 "~" H 7300 1850 50  0001 C CNN
-	1    7300 1850
-	0    -1   -1   0
-$EndComp
 Text Notes 10850 3400 2    50   ~ 0
 BUTTON PADS FOR FLIGHT CONTROL
-Text Label 9500 5800 2    50   ~ 0
-BTN_ROLL-
-Text Label 9500 5400 2    50   ~ 0
-BTN_ROLL+
-Text Label 9500 5000 2    50   ~ 0
-BTN_PITCH-
 Connection ~ 9900 5800
 Wire Wire Line
@@
 	1    0    0    -1
 $EndComp
-Text Label 9500 4600 2    50   ~ 0
-BTN_PITCH+
 Connection ~ 9900 5000
 Wire Wire Line
@@
 NoConn ~ 6250 4950
 $Comp
-L FEATHER_M0_BASIC_PROTO:FEATHER_M0_BASIC_PROTO U2
-U 1 1 602C87A2
-P 5400 2750
-F 0 "U2" H 5400 3917 50  0000 C CNN
-F 1 "FEATHER_M0_BASIC_PROTO" H 5400 3826 50  0000 C CNN
-F 2 "FEATHER_M0_BASIC_PROTO:FEATHER_M0_BASIC_PROTO" H 5400 2750 50  0001 L BNN
-F 3 "" H 5400 2750 50  0001 L BNN
-F 4 "Manufacturer Recommendation" H 5400 2750 50  0001 L BNN "STANDARD"
-F 5 "Adafruit" H 5400 2750 50  0001 L BNN "MANUFACTURER"
-	1    5400 2750
-	1    0    0    -1
-$EndComp
-Wire Wire Line
-	6700 1600 6700 1950
-Wire Wire Line
-	6700 1950 6600 1950
-Text Label 4200 3250 2    50   ~ 0
-GPS_TX
-Text Label 4200 3350 2    50   ~ 0
-GPS_RX
-Text Label 4200 3150 2    50   ~ 0
-MISO
-Text Label 4200 3050 2    50   ~ 0
-MOSI
-Text Label 4200 2950 2    50   ~ 0
-SCK
-Text Label 4200 2650 2    50   ~ 0
-BTN_A3
-NoConn ~ 4200 2050
-NoConn ~ 6600 2050
-NoConn ~ 4200 2250
-NoConn ~ 4200 2350
-Text Notes 4950 1350 0    50   ~ 0
-FEATHER M0 ADALOGGER
-$Comp
-L st_pat:Sharp_Display_4694 U4
+L st_pat_manual_ctrl_edits-rescue:Sharp_Display_4694-st_pat U4
 U 1 1 602ACB65
 P 8900 1750
@@
 NoConn ~ 9600 2200
 NoConn ~ 8650 2050
-Wire Wire Line
-	6850 1600 6850 1850
-Wire Wire Line
-	6850 1850 6600 1850
-Connection ~ 6850 1850
-$Comp
-L Device:LED D3
-U 1 1 60327137
-P 7000 2350
-F 0 "D3" H 6993 2095 50  0000 C CNN
-F 1 "GEN_BLU" H 6993 2186 50  0000 C CNN
-F 2 "LED_SMD:LED_1206_3216Metric_Pad1.42x1.75mm_HandSolder" H 7000 2350 50  0001 C CNN
-F 3 "~" H 7000 2350 50  0001 C CNN
-	1    7000 2350
-	-1   0    0    1
-$EndComp
-Wire Wire Line
-	6850 2350 6600 2350
-$Comp
-L Device:R_US R3
-U 1 1 60328426
-P 7300 2350
-F 0 "R3" V 7400 2350 50  0000 C CNN
-F 1 "100" V 7186 2350 50  0000 C CNN
-F 2 "Resistor_SMD:R_0805_2012Metric_Pad1.20x1.40mm_HandSolder" V 7340 2340 50  0001 C CNN
-F 3 "~" H 7300 2350 50  0001 C CNN
-	1    7300 2350
-	0    -1   -1   0
-$EndComp
-Wire Wire Line
-	7450 2750 7450 2350
-Connection ~ 7450 2350
-Wire Wire Line
-	7450 1850 7450 2350
-Wire Wire Line
-	6600 2550 6600 2350
-$Comp
-L st_pat:Telemetry_Breakout U5
+$Comp
+L st_pat_manual_ctrl_edits-rescue:Telemetry_Breakout-st_pat U5
 U 1 1 6032FDCF
 P 1700 4350
@@
 $EndComp
 $Comp
-L st_pat:Telemetry_Breakout U6
+L st_pat_manual_ctrl_edits-rescue:Telemetry_Breakout-st_pat U6
 U 1 1 603300CF
 P 3200 4350
@@
 Text Notes 2850 4200 0    50   ~ 0
 SRAD GPS RECEIVER
-Text Label 4200 2750 2    50   ~ 0
-COTS_RECV_CS_A4
-Text Label 4200 2850 2    50   ~ 0
-SRAD_RECV_CS_A5
 $Comp
 L power:GND #PWR013
@@
 Text Label 2850 5150 2    50   ~ 0
 MISO
-NoConn ~ 6600 2950
-Text Label 6600 2850 0    50   ~ 0
-CPS_CS_D10
-NoConn ~ 6600 3250
-NoConn ~ 6600 3350
-Text Notes 6950 3350 0    50   ~ 0
-P2_8 (D9) IS BATTERY MONITOR, DO NOT USE
 Text Notes 1700 1500 0    50   ~ 0
 25mA
-Text Notes 7050 1450 0    50   ~ 0
-Estimate 50mA
 Text Notes 8200 1750 0    50   ~ 0
 53uA
 $Comp
-L st_pat:GPS_Breakout_746 U1
+L st_pat_manual_ctrl_edits-rescue:GPS_Breakout_746-st_pat U1
 U 1 1 60E458B0
 P 2250 1750
@@
 Text Notes 7300 4150 0    50   ~ 0
 MANUAL <-> AUTOMATIC CONTROL
-Text Label 9500 4200 2    50   ~ 0
-BTN_YAW-
 Wire Wire Line
 	9900 4200 9900 4600
@@
 	1    0    0    -1
 $EndComp
-Text Label 9500 3800 2    50   ~ 0
-BTN_YAW+
 Connection ~ 9900 4200
 Wire Wire Line
@@
 Wire Wire Line
 	8750 5150 8750 5350
+$Comp
+L payload2022_custom:PIC18F26K83-canhw U?
+U 1 1 619850FD
+P 5500 2400
+F 0 "U?" H 5475 3315 50  0000 C CNN
+F 1 "PIC18F26K83-canhw" H 5475 3224 50  0000 C CNN
+F 2 "" H 5950 2400 50  0001 C CNN
+F 3 "" H 5950 2400 50  0001 C CNN
+	1    5500 2400
+	1    0    0    -1
+$EndComp
+$Comp
+L Connector:Conn_01x10_Female J?
+U 1 1 61988FD9
+P 4700 5000
+F 0 "J?" H 4728 4976 50  0000 L CNN
+F 1 "Conn_01x10_Female" H 4728 4885 50  0000 L CNN
+F 2 "" H 4700 5000 50  0001 C CNN
+F 3 "~" H 4700 5000 50  0001 C CNN
+	1    4700 5000
+	1    0    0    -1
+$EndComp
 Wire Notes Line
-	3450 2750 7700 2750
+	9050 6300 10950 6300
+Wire Notes Line
+	10950 6300 10950 3100
+Wire Notes Line
+	10950 3100 9150 3100
+Wire Notes Line
+	9150 3100 9150 6300
+Text Label 4500 4600 2    50   ~ 0
+BTN_YAW+
+Text Label 4500 4700 2    50   ~ 0
+BTN_YAW-
+Text Label 4500 4800 2    50   ~ 0
+BTN_PITCH+
+Text Label 4500 4900 2    50   ~ 0
+BTN_PITCH-
+Text Label 4500 5000 2    50   ~ 0
+BTN_ROLL+
+Text Label 4500 5100 2    50   ~ 0
+BTN_ROLL-
+Text Label 4800 4150 2    50   ~ 0
+BTN_PITCH+
+Text Label 4750 2750 2    50   ~ 0
+BTN_YAW+
+Text Label 4750 2850 2    50   ~ 0
+BTN_YAW-
+Text Label 4750 2950 2    50   ~ 0
+BTN_PITCH+
+Text Label 4750 3050 2    50   ~ 0
+BTN_PITCH-
+Text Label 6200 2850 0    50   ~ 0
+BTN_ROLL+
+Text Label 6200 2750 0    50   ~ 0
+BTN_ROLL-
 $EndSCHEMATC
