File: Manual-Controller/Manual-Controller.sch (KiCad schematic (older format))
At the start: 20 parts, among them J4 BATTERY, SW1 SW_PWR, SW2 BTN_RST, SW3 BTN, SW4 BTN, SW5 BTN, U1 GPS_Breakout_746, U2 FEATHER_M0_BASIC_PROTO, U4 Sharp_Display_4694

Commit message: added all manual controls
Parts:
- removed D3: GEN_BLU, LED_SMD:LED_1206_3216Metric_Pad1.42x1.75mm_HandSolder, symbol Device:LED
- removed R3: 100, Resistor_SMD:R_0805_2012Metric_Pad1.20x1.40mm_HandSolder, symbol Device:R_US
- added SW? (x2): BTN, Button_Switch_THT:SW_PUSH_6mm, symbol Switch:SW_Push
- added SW?: SW_AUTOPILOT, symbol Switch:SW_DIP_x01
- added SW?: SW_SAFETY, symbol Switch:SW_DIP_x01
- SW2: value BTN_RST -> BTN
- U?: symbol payload2022_custom:MCP2515-canhw -> Manual-Controller-rescue:MCP2515-canhw-payload2022_custom
Connections:
- net labels added: BTN_PITCH+, BTN_PITCH-, BTN_ROLL+, BTN_ROLL-, BTN_YAW+, BTN_YAW-, SW_AUTOPILOT, SW_SAFETY
- net labels removed: BTN_A1, BTN_A2, BTN_A3, CPS_CS_D10
- wire segments 44 -> 49
Other:
- note added: "AUTOMATIC/MANUAL CONTROL TOGGLE"
- note added: "FLIGHT CONTROL BUTTONS"
- note added: "SAFETY KILL SWITCH"
- note removed: "BUTTONS - ALL OF THEM HAVE INTERNAL PULLUP"
- moved on the sheet: J4, SW1, SW2, SW3, SW4, SW5

Commit message: assined footprints and fixed pins
Parts:
- added D2, D3, D4, D5, D6, D7: LED, LED_SMD:LED_0805_2012Metric_Pad1.15x1.40mm_HandSolder, symbol Device:LED
- C1, C2: renamed from C?; footprint (none) -> Capacitor_SMD:C_0805_2012Metric_Pad1.18x1.45mm_HandSolder
- J1: renamed from J?; footprint (none) -> TerminalBlock:TerminalBlock_bornier-2_P5.08mm
- R1: renamed from R?; footprint (none) -> Resistor_SMD:R_0805_2012Metric_Pad1.20x1.40mm_HandSolder
- SW2, SW3: renamed from SW?; footprint (none) -> Connector_JST:JST_XH_B2B-XH-AM_1x02_P2.50mm_Vertical
- U3: renamed from U?; footprint (none) -> payload2022_custom:mcp2562; symbol Manual-Controller-rescue:MCP2515-canhw-payload2022_custom -> Manual-Controller-rescue:MCP2515-canhw-payload2022_custom-Manual-Controller-rescue
- Y1: renamed from Y?; footprint (none) -> Crystal:Crystal_SMD_TXC_9HT11-2Pin_2.0x1.2mm_HandSoldering
- gave numbers to parts that had none: 3
- renumbered D2 to D1, J4 to J2, SW2 to SW4, SW3 to SW5, SW4 to SW6, SW5 to SW7, U1 to U2, U2 to U4, U4 to U5
Connections:
- wire segments 49 -> 55
Other:
- moved on the sheet: SW4, SW5, SW6, SW7, SW8, SW9

Commit message: finish schematic v1
Parts:
- removed D2, D3, D4, D5, D6, D7: LED, LED_SMD:LED_0805_2012Metric_Pad1.15x1.40mm_HandSolder, symbol Device:LED
- added SW10: BTN_RESET_EVERYTHING, Button_Switch_THT:SW_PUSH_6mm, symbol Switch:SW_Push
- added SW11: SW_DISP_ON, Connector_JST:JST_XH_B2B-XH-AM_1x02_P2.50mm_Vertical, symbol Switch:SW_DIP_x01
- U2: symbol st_pat-rescue:GPS_Breakout_746-st_pat -> Manual-Controller-rescue:GPS_Breakout_746-st_pat-st_pat-rescue
- U3: symbol Manual-Controller-rescue:MCP2515-canhw-payload2022_custom-Manual-Controller-rescue -> Manual-Controller-rescue:MCP2515-canhw-payload2022_custom-Manual-Controller-rescue-Manual-Controller-rescue
- U4: symbol st_pat-rescue:FEATHER_M0_BASIC_PROTO-FEATHER_M0_BASIC_PROTO -> Manual-Controller-rescue:FEATHER_M0_BASIC_PROTO-FEATHER_M0_BASIC_PROTO-st_pat-rescue
- U5: symbol st_pat-rescue:Sharp_Display_4694-st_pat -> Manual-Controller-rescue:Sharp_Display_4694-st_pat-st_pat-rescue
Connections:
- net labels added: XBEE_RESET
- net labels removed: SHARP_CS_D5, SHARP_DISP_D6
- wire segments 55 -> 66
- no-connect marks 21 -> 24
Other:
- moved on the sheet: SW4, SW5, SW6, SW7, SW8, SW9

Commit message: final schematic and lib consolidation
Parts:
- removed U3: MCP2515-canhw, payload2022_custom:mcp2562, symbol Manual-Controller-rescue:MCP2515-canhw-payload2022_custom-Manual-Controller-res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
- added R5: 5k, Resistor_SMD:R_0805_2012Metric_Pad1.20x1.40mm_HandSolder, symbol Device:R_US
- added U3: MCP2515_payload_22, payload2022_custom:MCP2515, symbol payload2022_custom:MCP2515_payload_22
- SW1: footprint st_pat:SW_Rocker_A22K1H-EA -> payload2022_custom:SW_Rocker_A22K1H-EA
- U2: footprint st_pat:GPS_Breakout_746 -> payload2022_custom:GPS_Breakout_746; symbol Manual-Controller-rescue:GPS_Breakout_746-st_pat-st_pat-rescue -> payload2022_custom:GPS_Breakout_746
- U4: footprint FEATHER_M0_BASIC_PROTO:FEATHER_M0_BASIC_PROTO -> payload2022_custom:FEATHER_M0_BASIC_PROTO; symbol Manual-Controller-rescue:FEATHER_M0_BASIC_PROTO-FEATHER_M0_BASIC_PROTO-st_pat-rescue -> payload2022_custom:FEATHER_M0_BASIC_PROTO-FEATHER_M0_BASIC_PROTO
- U5: footprint st_pat:Sharp_Display -> payload2022_custom:Sharp_Display; symbol Manual-Controller-rescue:Sharp_Display_4694-st_pat-st_pat-rescue -> payload2022_custom:Sharp_Display_4694
Connections:
- net +3V3: now also R5.1, U3.18 (VDD); no longer SW11.2, U5.6 (SCS)
- net BTN_PITCH+: now also U4.P1_9 (AIN4/VREFB/EINT/PA04); no longer U4.P2_12 (PA22/EINT/I2C/SDA)
- net BTN_PITCH-: now also U4.P1_8 (AIN5/EINT/PA05); no longer U4.P2_11 (PA23/EINT/I2C/SCL)
- net CAN_RX: now also U3.2 (RXCAN)
- net CAN_SCK: now also U4.P2_11 (PA23/EINT/I2C/SCL), U3.13 (SCK); no longer U4.P1_9 (AIN4/VREFB/EINT/PA04)
- net CAN_SD: now also U4.P2_9 (PA20/EINT/I2SSC), U3.15 (SO); no longer U4.P1_7 (AIN10/EINT/PB02)
- net CAN_SI: now also U4.P2_10 (PA15/EINT), U3.14 (SI); no longer U4.P1_8 (AIN5/EINT/PA05)
- net CAN_TX: now also U3.1 (TXCAN)
- net CAN_~CS: now also U4.P2_12 (PA22/EINT/I2C/SDA), U3.16 (~CS); no longer U4.P2_9 (PA20/EINT/I2SSC)
- net GND: now also U3.9 (VSS)
- net GPS_RX: now also U4.P2_6 (PA16/EINT/I2C); no longer U4.P1_2 (TX/I2SCK/EINT/PA10)
- net GPS_TX: now also U4.P2_7 (PA18/EINT); no longer U4.P1_3 (RX/I2SF0/EINT/PA11)
- net SW_AUTOPILOT: now also U4.P1_4 (MISO/I2C/PA12); no longer U4.P2_6 (PA16/EINT/I2C)
- net SW_SAFETY: now also U4.P1_7 (AIN10/EINT/PB02); no longer U4.P2_7 (PA18/EINT)
- net XBEE_RX: now also U4.P1_3 (RX/I2SF0/EINT/PA11); no longer U4.P1_4 (MISO/I2C/PA12)
- net XBEE_TX: now also U4.P1_2 (TX/I2SCK/EINT/PA10); no longer U4.P2_10 (PA15/EINT)
- net at R1.1: now also U3.17 (~RESET)
- net at C2.1, Y1.2: now also U3.8 (OSC1)
- net at C1.1, Y1.1: now also U3.7 (OSC2)
- new net: R5.2, SW11.2, U5.6 (SCS)
Changed lines of the file:
@@
 F 0 "SW1" H 4850 5385 50  0000 C CNN
 F 1 "SW_PWR" H 4850 5294 50  0000 C CNN
-F 2 "st_pat:SW_Rocker_A22K1H-EA" H 4850 5100 50  0001 C CNN
+F 2 "payload2022_custom:SW_Rocker_A22K1H-EA" H 4850 5100 50  0001 C CNN
 F 3 "https://www.nkkswitches.com/pdf/ARockers-1.pdf" H 4850 5100 50  0001 C CNN
 	1    4850 4900
@@
 NoConn ~ 5050 5000
 $Comp
-L Manual-Controller-rescue:FEATHER_M0_BASIC_PROTO-FEATHER_M0_BASIC_PROTO-st_pat-rescue U4
+L payload2022_custom:FEATHER_M0_BASIC_PROTO-FEATHER_M0_BASIC_PROTO U4
 U 1 1 602C87A2
 P 5400 2750
 F 0 "U4" H 5400 3917 50  0000 C CNN
 F 1 "FEATHER_M0_BASIC_PROTO" H 5400 3826 50  0000 C CNN
-F 2 "FEATHER_M0_BASIC_PROTO:FEATHER_M0_BASIC_PROTO" H 5400 2750 50  0001 L BNN
+F 2 "payload2022_custom:FEATHER_M0_BASIC_PROTO" H 5400 2750 50  0001 L BNN
 F 3 "" H 5400 2750 50  0001 L BNN
 F 4 "Manufacturer Recommendation" H 5400 2750 50  0001 L BNN "STANDARD"
@@
 Wire Wire Line
 	6700 1950 6600 1950
-Text Label 4200 3250 2    50   ~ 0
+Text Label 6600 2850 0    50   ~ 0
 GPS_TX
-Text Label 4200 3350 2    50   ~ 0
+Text Label 6600 2750 0    50   ~ 0
 GPS_RX
 NoConn ~ 4200 2050
@@
 FEATHER M0 ADALOGGER
 $Comp
-L Manual-Controller-rescue:Sharp_Display_4694-st_pat-st_pat-rescue U5
+L payload2022_custom:Sharp_Display_4694 U5
 U 1 1 602ACB65
 P 8900 1750
 F 0 "U5" H 9125 1865 50  0000 C CNN
 F 1 "Sharp_Display_4694" H 9125 1774 50  0000 C CNN
-F 2 "st_pat:Sharp_Display" H 8900 1750 50  0001 C CNN
+F 2 "payload2022_custom:Sharp_Display" H 8900 1750 50  0001 C CNN
 F 3 "" H 8900 1750 50  0001 C CNN
 	1    8900 1750
@@
 53uA
 $Comp
-L Manual-Controller-rescue:GPS_Breakout_746-st_pat-st_pat-rescue U2
+L payload2022_custom:GPS_Breakout_746 U2
 U 1 1 60E458B0
 P 2250 1750
 F 0 "U2" H 2250 1865 50  0000 C CNN
 F 1 "GPS_Breakout_746" H 2250 1774 50  0000 C CNN
-F 2 "st_pat:GPS_Breakout_746" H 2250 1750 50  0001 C CNN
+F 2 "payload2022_custom:GPS_Breakout_746" H 2250 1750 50  0001 C CNN
 F 3 "" H 2250 1750 50  0001 C CNN
 	1    2250 1750
@@
 Text Label 1650 4850 0    50   ~ 0
 XBEE_RX
-Text Label 4200 3150 2    50   ~ 0
+Text Label 4200 3250 2    50   ~ 0
 XBEE_RX
 $Comp
@@
 Wire Wire Line
 	1050 3800 1050 3750
-Text Label 6600 3150 0    50   ~ 0
+Text Label 4200 3350 2    50   ~ 0
 XBEE_TX
 Text Label 2750 5950 2    50   ~ 0
@@
 CAN_TX
 $Comp
-L Manual-Controller-rescue:MCP2515-canhw-payload2022_custom-Manual-Controller-rescue-Manual-Controller-rescue U3
-U 1 1 619F2F3F
-P 3300 6150
-F 0 "U3" H 3300 6615 50  0000 C CNN
-F 1 "MCP2515-canhw" H 3300 6524 50  0000 C CNN
-F 2 "payload2022_custom:mcp2562" H 3250 6150 50  0001 C CNN
-F 3 "" H 3250 6150 50  0001 C CNN
-	1    3300 6150
-	1    0    0    -1
-$EndComp
-$Comp
 L Device:C C2
 U 1 1 619E8E5F
@@
 CAN_SCK
 NoConn ~ 3850 6550
+Text Label 6600 3350 0    50   ~ 0
+CAN_~CS
 Text Label 6600 3050 0    50   ~ 0
-CAN_~CS
-Text Label 4200 2850 2    50   ~ 0
 CAN_SD
-Text Label 4200 2750 2    50   ~ 0
+Text Label 6600 3150 0    50   ~ 0
 CAN_SI
-Text Label 4200 2650 2    50   ~ 0
+Text Label 6600 3250 0    50   ~ 0
 CAN_SCK
 NoConn ~ 5350 -550
@@
 Text Label 4200 2550 2    50   ~ 0
 BTN_ROLL+
-Text Label 6600 3250 0    50   ~ 0
+Text Label 4200 2750 2    50   ~ 0
 BTN_PITCH-
-Text Label 6600 3350 0    50   ~ 0
+Text Label 4200 2650 2    50   ~ 0
 BTN_PITCH+
 Wire Wire Line
@@
 Text Label 5850 4700 2    50   ~ 0
 SW_AUTOPILOT
-Text Label 6600 2750 0    50   ~ 0
+Text Label 4200 3150 2    50   ~ 0
 SW_AUTOPILOT
-Text Label 6600 2850 0    50   ~ 0
+Text Label 4200 2850 2    50   ~ 0
 SW_SAFETY
 Wire Wire Line
@@
 L power:+3V3 #PWR034
 U 1 1 61CD4DE0
-P 10600 1950
-F 0 "#PWR034" H 10600 1800 50  0001 C CNN
-F 1 "+3V3" H 10615 2123 50  0000 C CNN
-F 2 "" H 10600 1950 50  0001 C CNN
-F 3 "" H 10600 1950 50  0001 C CNN
-	1    10600 1950
+P 10600 1650
+F 0 "#PWR034" H 10600 1500 50  0001 C CNN
+F 1 "+3V3" H 10615 1823 50  0000 C CNN
+F 2 "" H 10600 1650 50  0001 C CNN
+F 3 "" H 10600 1650 50  0001 C CNN
+	1    10600 1650
 	1    0    0    -1
 $EndComp
@@
 RST
 NoConn ~ 1650 5450
+$Comp
+L payload2022_custom:MCP2515_payload_22 U3
+U 1 1 61CBD3DB
+P 3300 6150
+F 0 "U3" H 3300 6615 50  0000 C CNN
+F 1 "MCP2515_payload_22" H 3300 6524 50  0000 C CNN
+F 2 "payload2022_custom:MCP2515" H 3250 6150 50  0001 C CNN
+F 3 "" H 3250 6150 50  0001 C CNN
+	1    3300 6150
+	1    0    0    -1
+$EndComp
+$Comp
+L Device:R_US R5
+U 1 1 61CBD530
+P 10600 1800
+F 0 "R5" H 10668 1846 50  0000 L CNN
+F 1 "5k" H 10668 1755 50  0000 L CNN
+F 2 "Resistor_SMD:R_0805_2012Metric_Pad1.20x1.40mm_HandSolder" V 10640 1790 50  0001 C CNN
+F 3 "~" H 10600 1800 50  0001 C CNN
+	1    10600 1800
+	1    0    0    -1
+$EndComp
 $EndSCHEMATC
